Commit message: Fix refactor and some audio changes. It may fail

File: ros2_ws/src/sancho_description/urdf/sancho_ranger.urdf (robot description, URDF)
Before this commit: robot ranger_mini_v3, 13 links, 12 joints
Links:
- removed link camera_link
- added link astra_camera_link; visual box size=0.05 0.05 0.05
- added link nose_camera_link; visual box size=0.03 0.03 0.03
Joints:
- added joint head_to_nose_camera: type fixed, parent head_link, child nose_camera_link, origin xyz=0.037 0.0 0.061 rpy=0 0 0
- joint base_to_camera: child camera_link -> astra_camera_link
